Commit message: I hope this urdf file isn't evil

File: onshape_conversion/converted_robot/robot.urdf (robot description, URDF)
Before this commit: robot onshape, 1 links, 0 joints
Links:
- removed link bevel_gear
- added link arm-cgb-assy, mass 7.9341350073740928295; collision mesh filename=package:///1.stl; collision mesh filename=package:///1.stl
