Commit message: Atempted urdf conversion with new cad that has joints

File: src/urdf_visualization/urdf/robot3.urdf (robot description, URDF)
Before this commit: robot onshape, 1 links, 0 joints
Links:
- link arm-cgb-assy: geometry collision mesh filename=package://urdf_visualization/urdf/meshes3/1.stl; collision mesh filename=package://urdf_visualization/urdf/meshes3/1.stl
