Commit message: Added new meshes for urdf visualization

File: src/urdf_visualization/urdf/robot.urdf (robot description, URDF)
Before this commit: robot onshape, 1 links, 0 joints
Links:
- removed link bevel_gear
- added link arm-cgb-assy, mass 7.9341350073740928295; collision mesh filename=package://urdf_visualization/urdf/meshes2/1.stl; collision mesh filename=package://urdf_visualization/urdf/meshes2/1.stl

Commit message: Added working new arm test urdf which is almost perfect except the rotation axis of each joint is a bit off relative to the links

File: src/urdf_visualization/urdf/robot.urdf (robot description, URDF)
Before this commit: robot onshape, 1 links, 0 joints
Links:
- removed link arm-cgb-assy
- added link base_link, mass 4.1507; collision mesh filename=package://urdf_visualization/urdf/meshes_2/base_link.STL; visual mesh filename=package://urdf_visualization/urdf/meshes_2/base_link.STL
- added link link_1, mass 5.297; collision mesh filename=package://urdf_visualization/urdf/meshes_2/link_1.STL; visual mesh filename=package://urdf_visualization/urdf/meshes_2/link_1.STL
- added link link_2, mass 0.69319; collision mesh filename=package://urdf_visualization/urdf/meshes_2/link_2.STL; visual mesh filename=package://urdf_visualization/urdf/meshes_2/link_2.STL
- added link link_3, mass 0.20963; collision mesh filename=package://urdf_visualization/urdf/meshes_2/link_3.STL; visual mesh filename=package://urdf_visualization/urdf/meshes_2/link_3.STL
Joints:
- added joint joint_1: type revolute, parent base_link, child link_1, origin xyz=0.022654 -0.16716 0.027062 rpy=0 0 3.1416, axis 0 1 0, limit lower=-1.5707 upper=1.5707 effort=63 velocity=10
- added joint joint_2: type revolute, parent link_1, child link_2, origin xyz=0.0127 0.11456 0.73061 rpy=6.2832 -1.5708 0, axis 0 1 0, limit lower=0 upper=3.1416 effort=33 velocity=10
- added joint joint_3: type revolute, parent link_2, child link_3, origin xyz=0 -0.012382 -0.5969 rpy=-1.5708 0 1.5708, axis 0 1 0, limit lower=0 upper=3.1416 effort=24 velocity=3

Commit message: CAD getting closer

File: src/urdf_visualization/urdf/robot.urdf (robot description, URDF)
Before this commit: robot arm_first_try, 4 links, 3 joints
Links:
- link base_link: mass 4.1507 -> 4.15068574213693
- link link_1: mass 5.297 -> 5.29698149295367
- link link_2: mass 0.69319 -> 0.693193740866267
- link link_3: mass 0.20963 -> 0.20963088398212
Joints:
- joint joint_1: axis 0 1 0 -> 0 -1 0; origin xyz=0.022654 -0.16716 0.027062 rpy=0 0 3.1416 -> xyz=0 0 0 rpy=0 0 0
- joint joint_2: limit lower=0 upper=3.1416 effort=33 velocity=10 -> lower=0 upper=3.1416 effort=30 velocity=10; origin xyz=0.0127 0.11456 0.73061 rpy=6.2832 -1.5708 0 -> xyz=0 0.11456 0.52669 rpy=0 0 0
- joint joint_3: axis 0 1 0 -> -1 0 0; origin xyz=0 -0.012382 -0.5969 rpy=-1.5708 0 1.5708 -> xyz=0.6223 0.14975 0.19121 rpy=0 0 0

Commit message: Reverting to closer urdf

File: src/urdf_visualization/urdf/robot.urdf (robot description, URDF)
Before this commit: robot arm, 4 links, 3 joints
Links:
- link base_link: mass 4.15068574213693 -> 4.1507
- link link_1: mass 5.29698149295367 -> 5.297
- link link_2: mass 0.693193740866267 -> 0.69319
- link link_3: mass 0.20963088398212 -> 0.20963
Joints:
- joint joint_1: axis 0 -1 0 -> 0 1 0; origin xyz=0 0 0 rpy=0 0 0 -> xyz=0.022654 -0.16716 0.027062 rpy=0 0 3.1416
- joint joint_2: limit lower=0 upper=3.1416 effort=30 velocity=10 -> lower=0 upper=3.1416 effort=33 velocity=10; origin xyz=0 0.11456 0.52669 rpy=0 0 0 -> xyz=0.0127 0.11456 0.73061 rpy=6.2832 -1.5708 0
- joint joint_3: axis -1 0 0 -> 0 1 0; origin xyz=0.6223 0.14975 0.19121 rpy=0 0 0 -> xyz=0 -0.012382 -0.5969 rpy=-1.5708 0 1.5708
