Commit message: Added directions for starting onshape converter in terminal

File: onshape_conversion/joint_1/robot.urdf (robot description, URDF)
Before this commit: robot onshape, 2 links, 1 joints
Links:
- removed link part_1
- removed link part_1__list_bssx4km84nfaeg_default
- added link link_arm__list_bssx4km84nfaeg_default, mass 0.35393517414960223855; collision mesh filename=package:///link_arm__list_bssx4km84nfaeg_default.stl; visual mesh filename=package:///link_arm__list_bssx4km84nfaeg_default.stl
- added link link_arm_hinge, mass 0; collision mesh filename=package:///link_arm_hinge.stl; visual mesh filename=package:///link_arm_hinge.stl
Joints:
- joint joint_1: child part_1__list_bssx4km84nfaeg_default -> link_arm__list_bssx4km84nfaeg_default; origin xyz=7.8901370748533069908e-22 0 -1.3781194271668015741e-21 rpy=1.570796326794896558 -0.34724469202426838654 3.141592653589793116 -> xyz=8.444870276581051764e-18 0 3.043347475119349751e-17 rpy=-1.570796326794896558 -0.9525144260775928462 3.2195723437558716655e-21; parent part_1 -> link_arm_hinge
