Commit message: Got joint error fixed but now relaxed_ik_rust giving error I think

File: src/relaxed_ik_ros2/relaxed_ik_core/configs/urdfs/model.urdf (robot description, URDF)
Before this commit: robot urdf_visualization/urdf, 7 links, 6 joints
Joints:
- removed joint wristRoll_link
- added joint wristRoll_joint: type revolute, parent carpus_link, child endEffector_link, origin xyz=0 0 0 rpy=0 0 0, axis 0 0 1, limit lower=0 upper=1.57 effort=50 velocity=1.5

Commit message: IK starting to work with new arm

File: src/relaxed_ik_ros2/relaxed_ik_core/configs/urdfs/model.urdf (robot description, URDF)
Before this commit: robot urdf_visualization/urdf, 7 links, 6 joints
Links:
- removed link carpus_link
- removed link endEffector_link
- removed link forearm_link
- removed link turntable_link
- removed link upperArm_link
- removed link wrist_link
- added link link_1, mass 5.2706; collision mesh filename=package://urdf_visualization/urdf/meshes_2/link_1.STL; visual mesh filename=package://urdf_visualization/urdf/meshes_2/link_1.STL
- added link link_2, mass 4; collision mesh filename=package://urdf_visualization/urdf/meshes_2/link_2.STL; visual mesh filename=package://urdf_visualization/urdf/meshes_2/link_2.STL
- added link link_3, mass 0.44193; collision mesh filename=package://urdf_visualization/urdf/meshes_2/link_3.STL; visual mesh filename=package://urdf_visualization/urdf/meshes_2/link_3.STL
- added link link_4, mass 0.4756; collision mesh filename=package://urdf_visualization/urdf/meshes_2/link_4.STL; visual mesh filename=package://urdf_visualization/urdf/meshes_2/link_4.STL
- link base_link: mass None -> 3; geometry collision mesh filename=package://urdf_visualization/urdf/meshes_2/base_link.STL; visual mesh filename=package://urdf_visualization/urdf/meshes_2/base_link.STL
Joints:
- removed joint elbowPitch_joint
- removed joint elbowRoll_joint
- removed joint shoulder_joint
- removed joint turntable_joint
- removed joint wristPitch_joint
- removed joint wristRoll_joint
- added joint joint_1: type revolute, parent base_link, child link_1, origin xyz=0 0 0 rpy=0 0 0, axis 0 -1 0, limit lower=-1.5707 upper=1.5707 effort=63 velocity=10
- added joint joint_2: type revolute, parent link_1, child link_2, origin xyz=0 0.11456 0.69567 rpy=0 0 0, axis 0 1 0, limit lower=-1.60 upper=3.1416 effort=30 velocity=10
- added joint joint_3: type revolute, parent link_2, child link_3, origin xyz=-0.68187 -0.14975 0 rpy=3.1416 -1.5708 1.5708, axis 0 0 1, limit lower=-1.6 upper=1.6 effort=24 velocity=3
- added joint joint_4: type revolute, parent link_3, child link_4, origin xyz=0 -0.0381 0 rpy=0 0 0, axis 0 -1 0, limit lower=-3.14 upper=3.14 effort=0 velocity=0

File: src/urdf_visualization/urdf/robot.urdf (robot description, URDF)
Before this commit: robot arm_first_try, 4 links, 3 joints
Links:
- added link link_4, mass 0.4756; collision mesh filename=package://urdf_visualization/urdf/meshes_2/link_4.STL; visual mesh filename=package://urdf_visualization/urdf/meshes_2/link_4.STL
- link base_link: mass 4.1507 -> 3
- link link_1: mass 5.297 -> 5.2706
- link link_2: mass 0.69319 -> 4
- link link_3: mass 0.20963 -> 0.44193
Joints:
- added joint joint_4: type revolute, parent link_3, child link_4, origin xyz=0 -0.0381 0 rpy=0 0 0, axis 0 -1 0, limit lower=-3.14 upper=3.14 effort=0 velocity=0
- joint joint_1: axis 0 1 0 -> 0 -1 0; origin xyz=0.022654 -0.16716 0.027062 rpy=0 0 3.1416 -> xyz=0 0 0 rpy=0 0 0
- joint joint_2: limit lower=0 upper=3.1416 effort=33 velocity=10 -> lower=-1.60 upper=3.1416 effort=30 velocity=10; origin xyz=0.0127 0.11456 0.73061 rpy=6.2832 -1.5708 0 -> xyz=0 0.11456 0.69567 rpy=0 0 0
- joint joint_3: axis 0 1 0 -> 0 0 1; limit lower=0 upper=3.1416 effort=24 velocity=3 -> lower=-1.6 upper=1.6 effort=24 velocity=3; origin xyz=0 -0.012382 -0.5969 rpy=-1.5708 0 1.5708 -> xyz=-0.68187 -0.14975 0 rpy=3.1416 -1.5708 1.5708
