Commit message: Working on cleaning up the arm relaxed IK

File: src/relaxed_ik_ros2/relaxed_ik_core/configs/urdfs/urc_arm.urdf (robot description, URDF)
Before this commit: robot robot_arm_urdf_complete, 5 links, 4 joints
Links:
- link base_link: geometry collision mesh filename=package://urdf_visualization/meshes/base_link.STL; visual mesh filename=package://urdf_visualization/meshes/base_link.STL
- link link_1: geometry collision mesh filename=package://urdf_visualization/meshes/link_1.STL; visual mesh filename=package://urdf_visualization/meshes/link_1.STL
- link link_2: geometry collision mesh filename=package://urdf_visualization/meshes/link_2.STL; visual mesh filename=package://urdf_visualization/meshes/link_2.STL
- link link_3: geometry collision mesh filename=package://urdf_visualization/meshes/link_3.STL; visual mesh filename=package://urdf_visualization/meshes/link_3.STL
- link link_4: geometry collision mesh filename=package://urdf_visualization/meshes/link_4.STL; visual mesh filename=package://urdf_visualization/meshes/link_4.STL

Commit message: Further cleanup and remaining

File: src/relaxed_ik_ros2/relaxed_ik_core/configs/urdfs/urc_arm.urdf (robot description, URDF)
Before this commit: robot robot_arm_urdf_complete, 5 links, 4 joints
Links:
- link base_link: geometry collision mesh filename=package://arm_ik/meshes/base_link.STL; visual mesh filename=package://arm_ik/meshes/base_link.STL
- link link_1: geometry collision mesh filename=package://arm_ik/meshes/link_1.STL; visual mesh filename=package://arm_ik/meshes/link_1.STL
- link link_2: geometry collision mesh filename=package://arm_ik/meshes/link_2.STL; visual mesh filename=package://arm_ik/meshes/link_2.STL
- link link_3: geometry collision mesh filename=package://arm_ik/meshes/link_3.STL; visual mesh filename=package://arm_ik/meshes/link_3.STL
- link link_4: geometry collision mesh filename=package://arm_ik/meshes/link_4.STL; visual mesh filename=package://arm_ik/meshes/link_4.STL
