Commit message: IK simulation working better for controlling arm

File: src/relaxed_ik_ros2/relaxed_ik_core/configs/urdfs/arm_urdf.urdf (robot description, URDF)
Before this commit: robot arm2_urdf, 5 links, 4 joints
Links:
- link link_1: mass 5.22444424208244 -> 5.22444423373266
- link link_2: mass 0.811667223175114 -> 0.811667223501401
Joints:
- joint joint_2: limit lower=-1.5707 upper=6.2802 effort=30 velocity=10 -> lower=4.75238898038 upper=7.8539 effort=30 velocity=10; origin xyz=0 0.11456 0.5716 rpy=0 0 0 -> xyz=0.010339 0.11456 0.57151 rpy=0 0 0
- joint joint_3: axis 0 0 1 -> 0 0 -1; limit lower=-1.5707 upper=1.5707 effort=24 velocity=3 -> lower=-2.3561 upper=2.3561 effort=24 velocity=3; origin xyz=-0.50776 -0.14975 0 rpy=3.1416 -1.5708 1.5708 -> xyz=-0.50747 -0.14975 0.017051 rpy=1.5708 -1.5372 0
- joint joint_4: axis 0 -1 0 -> 0.0 -1.0 0; origin xyz=0 -0.0381 0 rpy=0 0 0 -> xyz=0 0 0 rpy=3.1416 0 0.033598

Commit message: Nico stuff

File: src/relaxed_ik_ros2/relaxed_ik_core/configs/urdfs/arm_urdf.urdf (robot description, URDF)
Before this commit: robot arm_ik, 5 links, 4 joints
Joints:
- joint joint_3: limit lower=-2.3561 upper=2.3561 effort=24 velocity=3 -> lower=-1.9561 upper=2.2561 effort=24 velocity=3

File: src/relaxed_ik_ros2/relaxed_ik_core/configs/urdfs/urc_arm.urdf (robot description, URDF)
Before this commit: robot robot_arm_urdf_complete, 5 links, 4 joints
Joints:
- joint joint_3: limit lower=-1.6 upper=1.6 effort=24 velocity=3 -> lower=-1.6 upper=1.1 effort=24 velocity=3
